File: Kicad/Mowgli/HC245.sch (KiCad schematic (older format))
At the start: 4 parts, among them P1 Isolate

Commit message: updated Kicad with Charge/Battery Circuit
Parts:
- IC? (x2): symbol HC254:SN74ABT245BMDBREP -> Mowgli-rescue:SN74ABT245BMDBREP-HC254
Changed lines of the file:
@@
 $Descr A4 11693 8268
 encoding utf-8
-Sheet 5 9
+Sheet 9 10
 Title "Project Mowgli"
 Date "2022-05-22"
@@
 $EndDescr
 $Comp
-L HC254:SN74ABT245BMDBREP IC?
+L Mowgli-rescue:SN74ABT245BMDBREP-HC254 IC?
 U 1 1 628B1A7E
 P 4600 2100
+AR Path="/628B1A7E" Ref="IC?"  Part="1"
+AR Path="/628B14E1/628B1A7E" Ref="IC?"  Part="1"
 F 0 "IC?" H 5100 2365 50  0000 C CNN
 F 1 "74HC245 (from STM)" H 5100 2274 50  0000 C CNN
@@
 $EndComp
 $Comp
-L HC254:SN74ABT245BMDBREP IC?
+L Mowgli-rescue:SN74ABT245BMDBREP-HC254 IC?
 U 1 1 628B4641
 P 4600 3750
+AR Path="/628B4641" Ref="IC?"  Part="1"
+AR Path="/628B14E1/628B4641" Ref="IC?"  Part="1"
 F 0 "IC?" H 5100 4015 50  0000 C CNN
 F 1 "74HC254 (to STM)" H 5100 3924 50  0000 C CNN

Commit message: updated kicad
Other:
- note added: "Jumper"
Changed lines of the file:
@@
 Wire Wire Line
 	4600 4250 4100 4250
+Text Notes 4950 1350 0    118  ~ 0
+Jumper
 $EndSCHEMATC
