File: Kicad/Mowgli/J18 (Red Connector).sch (KiCad schematic (older format))
At the start: 1 part, among them J18 (Red Connector)

Commit message: added J18 SPI3 pins
Connections:
- net J18_Pin_3_SPI3_DI: now reaches J18.3 (Pin_3)
- net J18_Pin_4_SPI3_DO: now reaches J18.4 (Pin_4)
- net J18_Pin_5_SPI3_CLK: now reaches J18.5 (Pin_5)
Other:
- note added: "SPI 3"
Changed lines of the file:
@@
 $Descr A4 11693 8268
 encoding utf-8
-Sheet 5 10
+Sheet 5 11
 Title "Project Mowgli"
 Date "2022-05-22"
@@
 L power:GND #PWR0109
 U 1 1 629291C3
-P 5450 3850
-F 0 "#PWR0109" H 5450 3600 50  0001 C CNN
-F 1 "GND" H 5455 3677 50  0000 C CNN
-F 2 "" H 5450 3850 50  0001 C CNN
-F 3 "" H 5450 3850 50  0001 C CNN
-	1    5450 3850
+P 6250 3750
+F 0 "#PWR0109" H 6250 3500 50  0001 C CNN
+F 1 "GND" H 6255 3577 50  0000 C CNN
+F 2 "" H 6250 3750 50  0001 C CNN
+F 3 "" H 6250 3750 50  0001 C CNN
+	1    6250 3750
 	1    0    0    -1
 $EndComp
-Wire Wire Line
-	5450 3850 5450 3750
-Wire Wire Line
-	5450 3750 5200 3750
 Text HLabel 6250 3050 2    50   UnSpc ~ 0
 J18_Pin_2
@@
 Wire Wire Line
 	5200 3450 6250 3450
+Text Notes 7100 3300 0    50   Italic 10
+SPI 3
+Wire Wire Line
+	6250 3150 5200 3150
+Wire Wire Line
+	5200 3250 6250 3250
+Wire Wire Line
+	6250 3350 5200 3350
+Text HLabel 6250 3350 2    50   Input ~ 0
+J18_Pin_5_SPI3_CLK
+Text HLabel 6250 3250 2    50   Input ~ 0
+J18_Pin_4_SPI3_DO
+Text HLabel 6250 3150 2    50   Output ~ 0
+J18_Pin_3_SPI3_DI
+Wire Wire Line
+	5200 3750 6250 3750
 $EndSCHEMATC
