File: Kicad/Mowgli/J6 (Control Panel).sch (KiCad schematic (older format))
At the start: 1 part, among them J6 Control Panel

Commit message: updated Kicad with Charge/Battery Circuit
Parts:
- removed J6: Control Panel, symbol Connector:Conn_01x16_Male
- added J6: Contrl Panel, symbol Connector_Generic_MountingPin:Conn_02x08_Odd_Even_MountingPin
Changed lines of the file:
@@
 $Descr A4 11693 8268
 encoding utf-8
-Sheet 7 9
+Sheet 6 10
 Title "Project Mowgli"
 Date "2022-05-22"
@@
 Comment4 ""
 $EndDescr
+Text HLabel 5350 3100 0    50   Input ~ 0
+J6_Pin_1
+Text HLabel 5350 3200 0    50   Output ~ 0
+J6_Pin_3
 $Comp
-L Connector:Conn_01x16_Male J6
-U 1 1 629324E6
-P 4900 2850
-F 0 "J6" H 5008 3731 50  0000 C CNN
-F 1 "Control Panel" H 5008 3640 50  0000 C CNN
-F 2 "" H 4900 2850 50  0001 C CNN
-F 3 "~" H 4900 2850 50  0001 C CNN
-	1    4900 2850
+L Connector_Generic_MountingPin:Conn_02x08_Odd_Even_MountingPin J6
+U 1 1 628D511C
+P 5850 3400
+F 0 "J6" H 5900 3917 50  0000 C CNN
+F 1 "Contrl Panel" H 5900 3826 50  0000 C CNN
+F 2 "" H 5850 3400 50  0001 C CNN
+F 3 "~" H 5850 3400 50  0001 C CNN
+	1    5850 3400
 	1    0    0    -1
 $EndComp
-Text HLabel 5800 2950 2    50   UnSpc ~ 0
+Wire Wire Line
+	5650 3100 5350 3100
+Wire Wire Line
+	5650 3200 5350 3200
+Text Notes 4450 3150 0    50   ~ 0
+USART 1 (TX)
+Text Notes 4450 3250 0    50   ~ 0
+USART 1 (RX)
+Text Notes 4450 3250 0    50   ~ 0
+USART 1 (RX)
+Text HLabel 5350 3500 0    50   UnSpc ~ 0
 J6_Pin_9
 Wire Wire Line
-	5800 2950 5100 2950
-Text HLabel 5800 2150 2    50   Input ~ 0
-J6_Pin_1
-Text HLabel 5800 2350 2    50   Output ~ 0
-J6_Pin_3
-Wire Wire Line
-	5800 2150 5100 2150
-Wire Wire Line
-	5800 2350 5100 2350
-Text Notes 6200 2400 0    50   ~ 0
-USART 1 (RX)
-Text Notes 6200 2200 0    50   ~ 0
-USART 1 (TX)
+	5650 3500 5350 3500
 $EndSCHEMATC

Commit message: added more details to panel J6 connector, and reversed rain sensor (STM32 PE2)
Parts:
- removed J6: Contrl Panel, symbol Connector_Generic_MountingPin:Conn_02x08_Odd_Even_MountingPin
- added C17, C3, C4, C5, C6, C8: C, symbol Device:C
- added FB1: Ferrite_Bead, symbol Device:Ferrite_Bead
- added J6: Control Panel, symbol Connector_Generic:Conn_02x08_Odd_Even
- added JP1: Rain Sensor, symbol Connector:Conn_01x02_Male
- added JP4: Sensor Harness, symbol Connector:Conn_01x12_Male
- added Q2, Q4, Q5, Q6: NMOS_G15, symbol Device:Q_NMOS_SGD
- added R27: 200, symbol Device:R
- added R33: 0, symbol Device:R
- added R50, R61, R74, R83: 10k, symbol Device:R
- added R55, R64, R78, R86: 100k, symbol Device:R
- added SW3: PLAY, symbol Switch:SW_Push
- added U3: AMS1117-3.3, Package_TO_SOT_SMD:SOT-223-3_TabPin2, symbol Regulator_Linear:AMS1117-3.3
Connections:
- net labels added: +3.3V, +5V, GND, J6_Pin_10_Wheel_blue, J6_Pin_11_RainSensor, J6_Pin_14_Stop_yellow, J6_Pin_16_Wheel_red, J6_Pin_4_PLAY, J6_Pin_6_Stop_white
- wire segments 3 -> 126
Other:
- note added: "5V Supply"
- note added: "Rain Sensor"
- note added: "Stop Hall (white)"
- note added: "Stop Hall (yellow)"
- note added: "Wheel Lift Hall (blue)"
- note added: "Wheel Lift Hall (red)"

Commit message: reversed mechanical tilt and accelerometer circuit
Connections:
- net labels added: J6_Pin_15,13,12,8,7_GND
- wire segments 126 -> 128
Changed lines of the file:
@@
 $Descr A4 11693 8268
 encoding utf-8
-Sheet 11 14
+Sheet 10 14
 Title "Project Mowgli"
 Date "2022-05-22"
@@
 	4750 5050 4000 5050
 Wire Wire Line
-	4000 4700 4000 5050
+	4000 4700 4000 4900
 Connection ~ 4750 4500
 Connection ~ 4000 5050
@@
 Wire Wire Line
 	1550 4500 4100 4500
+Text HLabel 3800 4900 0    50   Output ~ 0
+J6_Pin_15,13,12,8,7_GND
+Wire Wire Line
+	3800 4900 4000 4900
+Connection ~ 4000 4900
+Wire Wire Line
+	4000 4900 4000 5050
 $EndSCHEMATC

Commit message: panel updates
Parts:
- added SW1: CLOCK, symbol Switch:SW_Push
Connections:
- net labels added: J6_Pin_2_CLOCK
- wire segments 128 -> 134
Changed lines of the file:
@@
 L power:GND #PWR?
 U 1 1 629F7C3E
-P 4000 5650
-F 0 "#PWR?" H 4000 5400 50  0001 C CNN
-F 1 "GND" H 4005 5477 50  0000 C CNN
-F 2 "" H 4000 5650 50  0001 C CNN
-F 3 "" H 4000 5650 50  0001 C CNN
-	1    4000 5650
+P 4000 6200
+F 0 "#PWR?" H 4000 5950 50  0001 C CNN
+F 1 "GND" H 4005 6027 50  0000 C CNN
+F 2 "" H 4000 6200 50  0001 C CNN
+F 3 "" H 4000 6200 50  0001 C CNN
+	1    4000 6200
 	1    0    0    -1
 $EndComp
@@
 	4250 5450 4000 5450
 Connection ~ 4000 5450
-Wire Wire Line
-	4000 5450 4000 5650
 Text HLabel 5100 4950 3    50   Output ~ 0
 J6_Pin_10_Wheel_blue
@@
 	6650 4700 6650 4950
 Connection ~ 6650 4700
-Text HLabel 4850 5750 3    50   Output ~ 0
+Text HLabel 4850 6250 3    50   Output ~ 0
 J6_Pin_4_PLAY
-Wire Wire Line
-	4850 5450 4850 5750
 Connection ~ 4850 5450
 Text HLabel 1550 4350 1    50   Output ~ 0
@@
 Wire Wire Line
 	4000 4900 4000 5050
+Text HLabel 4950 6250 3    50   Output ~ 0
+J6_Pin_2_CLOCK
+Wire Wire Line
+	4600 4000 4950 4000
+Wire Wire Line
+	4850 5450 4850 6250
+$Comp
+L Switch:SW_Push SW1
+U 1 1 62CD5D52
+P 4450 5950
+F 0 "SW1" H 4450 5765 50  0000 C CNN
+F 1 "CLOCK" H 4450 5856 50  0000 C CNN
+F 2 "" H 4450 6150 50  0001 C CNN
+F 3 "~" H 4450 6150 50  0001 C CNN
+	1    4450 5950
+	-1   0    0    1
+$EndComp
+Wire Wire Line
+	4950 4000 4950 5950
+Wire Wire Line
+	4250 5950 4000 5950
+Connection ~ 4000 5950
+Wire Wire Line
+	4000 5950 4000 6200
+Wire Wire Line
+	4000 5450 4000 5950
+Wire Wire Line
+	4650 5950 4950 5950
+Connection ~ 4950 5950
+Wire Wire Line
+	4950 5950 4950 6250
 $EndSCHEMATC
